File: pcb/lasko_ir_remote.kicad_pcb (KiCad board)
At the start: 2 copper layers, 27 x 54.5 mm, 16 parts, among them J1 UPDI, Q1 MMBT2222A, SW1 SW_Push, SW2 SW_Push, SW3 SW_Push, SW4 SW_Push, U1 ATtiny212-SS

Commit message: pcb layout
Parts:
- added BT1: AAA, pl_battery:BK-82_AAA_1Cell, B.Cu at (156.8, 114.3)
- added BT2: AAA, pl_battery:BK-82_AAA_1Cell, B.Cu at (143.2, 114.3)
- moved H2 42.0 mm to (133.5, 136.5)
- moved H3 42.0 mm to (166.5, 136.5)
- moved J1 27.0 mm to (168.0, 68.8)
- moved D2 14.8 mm to (162.2, 86.8)
- moved H1 6.50 mm to (133.5, 47.5)
- moved H4 6.50 mm to (166.5, 47.5)
- moved R1 5.62 mm to (160.8, 48.0), turned to 180 degrees
- moved C1 5.27 mm to (158.6, 67.5)
- moved U1 4.75 mm to (163.2, 70.0)
- moved Q1 4.47 mm to (156.2, 46.8), turned to 90 degrees
- moved R2 2.77 mm to (144.8, 48.2), turned to 90 degrees
Routing:
- net Net-(BT1--): track 0.00 -> 33.0 mm
- net GND: track 0.00 -> 26.0 mm
- net /~{RESET}: track 21.9 -> 5.84 mm
- net /BUTTON_2: track 8.44 -> 13.2 mm
- net /BUTTON_1: track 6.86 -> 11.5 mm
- net /BUTTON_3: track 19.3 -> 23.4 mm
- net /BUTTON_0: track 16.2 -> 20.0 mm
- net VCC: track 78.9 -> 76.5 mm
- net /IR_CTRL: track 19.1 -> 21.0 mm
- net Net-(Q1-B): track 4.29 -> 2.68 mm
- net Net-(D1-K): track 3.50 -> 5.03 mm
- net Net-(D1-A): track 3.69 -> 4.76 mm
- added copper zone on B.Cu, net Net-(BT1--)
- added copper zone on B.Cu, net VCC
Other:
- board size 27 x 54.5 mm -> 40 x 96 mm
